Commit message: Proper configuration of differential drive odom

File: description/diffRobotBasic.urdf.xacro (robot description, xacro)
@@ -1,10 +1,4 @@
 <robot xmlns:xacro="http://www.ros.org/wiki/xacro" name="MyRobot">
     <xacro:include filename="baseInertial.xacro" />
-    <link name="dummy_link">
-    </link>
-    <joint name="dummy_join" type="fixed">
-        <parent link="dummy_link"/>
-        <child link="base_link"/>
-    </joint>
     <link name="base_link">
         <xacro:basic_box mass="1." x="1." y="0.7" z="0.2" r="1" g="0" b="0">
@@ -54,4 +48,5 @@
         <child link="head_link"/>
     </joint>
+<!--
     <gazebo>
         <plugin name="gazebo_ros_joint_state_publisher" filename="libgazebo_ros_joint_state_publisher.so">
@@ -61,4 +56,5 @@
         </plugin>
     </gazebo>
+-->
     <gazebo reference="base_link">
         <material> Gazebo/Red </material>
@@ -94,5 +90,5 @@
             <publish_wheel_tf>true</publish_wheel_tf>
             <odometry_topic>odom</odometry_topic>
-            <odometry_frame>base_link</odometry_frame>
+            <odometry_frame>odom</odometry_frame>
             <robot_base_frame>base_link</robot_base_frame>
         </plugin>

Commit message: Added Lidar

File: description/diffRobotBasic.urdf.xacro (robot description, xacro)
@@ -31,4 +31,9 @@
         </xacro:basic_box>
     </link>
+    <link name="lidar_link">
+        <xacro:basic_cylinder mass=".1" radius=".1" length=".2" r="0" g="1" b="1">
+            <origin xyz="0.0 0.0 -0.05" rpy="0 0 0.0"/>
+        </xacro:basic_cylinder>
+    </link>
     <joint name="base_wheelR_joint" type="continuous">
         <origin xyz="0.0 -0.4 0.0" rpy="0.0 0.0 0.0"/>
@@ -48,13 +53,9 @@
         <child link="head_link"/>
     </joint>
-<!--
-    <gazebo>
-        <plugin name="gazebo_ros_joint_state_publisher" filename="libgazebo_ros_joint_state_publisher.so">
-            <update_rate>1</update_rate>
-            <joint_name>base_wheelL_joint</joint_name>
-            <joint_name>base_wheelR_joint</joint_name>
-        </plugin>
-    </gazebo>
--->
+    <joint name="base_lidar_link" type="fixed">
+        <origin xyz="0.60 0.0 0.25" rpy="0.0 0.0 0.0"/>
+        <parent link="base_link"/>
+        <child link="lidar_link"/>
+    </joint>
     <gazebo reference="base_link">
         <material> Gazebo/Red </material>
@@ -94,3 +95,33 @@
         </plugin>
     </gazebo>
+    <gazebo reference="lidar_link">
+        <sensor type="gpu_ray" name="lidar_sensor">
+            <ray>
+                <scan>
+                    <horizontal>
+                        <samples>300</samples>
+                        <resolution>1</resolution>
+                        <min_angle>-3.141592</min_angle>
+                        <max_angle>3.141592</max_angle>
+                    </horizontal>
+                </scan>
+                <range>
+                    <min>0.10</min>
+                    <max>10.0</max>
+                    <resolution>0.01</resolution>
+                </range>
+                <noise>
+                    <type>gaussian</type>
+                    <mean>0.0</mean>
+                    <stddev>0.01</stddev>
+                </noise>
+            </ray>
+            <update_rate>5</update_rate>
+            <visualize>true</visualize>
+            <plugin name="lidar" filename="libgazebo_ros_ray_sensor.so">
+                <output_type>sensor_msgs/PointCloud2</output_type>
+                <frame_name>lidar_link</frame_name>
+            </plugin>
+        </sensor>
+    </gazebo>
 </robot>

Commit message: Added IMU

File: description/diffRobotBasic.urdf.xacro (robot description, xacro)
@@ -36,4 +36,9 @@
         </xacro:basic_cylinder>
     </link>
+    <link name="IMU_link">
+        <xacro:basic_cylinder mass=".1" radius=".1" length=".05" r="0" g="1" b="1">
+            <origin xyz="0.0 0.0 -0.0" rpy="0 0 0.0"/>
+        </xacro:basic_cylinder>
+    </link>
     <joint name="base_wheelR_joint" type="continuous">
         <origin xyz="0.0 -0.4 0.0" rpy="0.0 0.0 0.0"/>
@@ -57,4 +62,9 @@
         <parent link="base_link"/>
         <child link="lidar_link"/>
+    </joint>
+    <joint name="base_IMU_link" type="fixed">
+        <origin xyz="0.0 0.0 0.125" rpy="0.0 0.0 0.0"/>
+        <parent link="base_link"/>
+        <child link="IMU_link"/>
     </joint>
     <gazebo reference="base_link">
@@ -125,3 +135,71 @@
         </sensor>
     </gazebo>
+    <gazebo reference="IMU_link">
+        <sensor name="imu_sensor" type="imu">
+        <plugin filename="libgazebo_ros_imu_sensor.so" name="imu_plugin">
+            <ros>
+                <namespace>/imu</namespace>
+                <remapping>~/out:=out</remapping>
+            </ros>
+            <initial_orientation_as_reference>false</initial_orientation_as_reference>
+            </plugin>
+            <always_on>true</always_on>
+            <update_rate>100</update_rate>
+            <visualize>true</visualize>
+            <imu>
+            <angular_velocity>
+                <x>
+                <noise type="gaussian">
+                    <mean>0.0</mean>
+                    <stddev>2e-4</stddev>
+                    <bias_mean>0.0000075</bias_mean>
+                    <bias_stddev>0.0000008</bias_stddev>
+                </noise>
+                </x>
+                <y>
+                <noise type="gaussian">
+                    <mean>0.0</mean>
+                    <stddev>2e-4</stddev>
+                    <bias_mean>0.0000075</bias_mean>
+                    <bias_stddev>0.0000008</bias_stddev>
+                </noise>
+                </y>
+                <z>
+                <noise type="gaussian">
+                    <mean>0.0</mean>
+                    <stddev>2e-4</stddev>
+                    <bias_mean>0.0000075</bias_mean>
+                    <bias_stddev>0.0000008</bias_stddev>
+                </noise>
+                </z>
+            </angular_velocity>
+            <linear_acceleration>
+                <x>
+                <noise type="gaussian">
+                    <mean>0.0</mean>
+                    <stddev>1.7e-2</stddev>
+                    <bias_mean>0.1</bias_mean>
+                    <bias_stddev>0.001</bias_stddev>
+                </noise>
+                </x>
+                <y>
+                <noise type="gaussian">
+                    <mean>0.0</mean>
+                    <stddev>1.7e-2</stddev>
+                    <bias_mean>0.1</bias_mean>
+                    <bias_stddev>0.001</bias_stddev>
+                </noise>
+                </y>
+                <z>
+                <noise type="gaussian">
+                    <mean>0.0</mean>
+                    <stddev>1.7e-2</stddev>
+                    <bias_mean>0.1</bias_mean>
+                    <bias_stddev>0.001</bias_stddev>
+                </noise>
+                </z>
+            </linear_acceleration>
+            </imu>
+        </sensor>
+    </gazebo>
 </robot>
